File: MatrixBuddyPCB/MatrixBuddyPCB.kicad_sch (KiCad schematic)
At the start: 18 parts, among them J1 Conn_01x08_Pin, J2 Conn_01x08_Socket, J3 BATT Connector, Q1 Q_PMOS_GSD, SW1 SW_Push, SW2 SW_Push, SW3 SW_Push, U1 MAX7221xWG, U2 4104, U3 SeeeduinoXIAO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

Commit message: Bugfixing ahead of first production batch.
Connections:
- no-connect marks 5 -> 14
Other:
- note added: "MAJOR ERROR: MOSI and CS lines to 4104 swapped CORRECT PINMAP: CS - 10 MOSI - 9 SCK - 8"
Changed lines of the file:
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@@
   (no_connect (at 210.82 95.25))
   (no_connect (at 210.82 87.63))
+  (no_connect (at 209.55 146.05))
+  (no_connect (at 228.6 160.02))
+  (no_connect (at 229.87 115.57))
+  (no_connect (at 233.68 115.57))
+  (no_connect (at 226.06 115.57))
   (no_connect (at 210.82 97.79))
   (no_connect (at 210.82 82.55))
+  (no_connect (at 233.68 160.02))
+  (no_connect (at 209.55 149.86))
+  (no_connect (at 237.49 115.57))
   (no_connect (at 210.82 92.71))
+  (no_connect (at 251.46 149.86))
   (wire (pts (xy 132.08 97.79) (xy 199.39 97.79))
     (stroke (width 0) (type default))
@@
     (effects (font (size 1.27 1.27)) (justify left top))
   )
+  (text "MAJOR ERROR:\nMOSI and CS lines \nto 4104 swapped\nCORRECT PINMAP:\nCS   - 10\nMOSI -  9\nSCK  -  8"
+    (at 290.83 109.22 0)
+    (effects (font (size 2.54 2.54) (thickness 0.254) bold (color 190 2 19 1)) (justify left bottom))
+  )
   (label "BUTT1_B2" (at 133.35 92.71 0) (fields_autoplaced)
